Commit message: got rear wheels tfs

File: src/my_robot_gazebo/urdf/materials.xacro (robot description, xacro)
@@ -1,35 +1,25 @@
-<?xml version="1.0" ?>
-<!--  xacro macros for robot materials.
- -->
-<robot name="materials" xmlns:xacro="http://wiki.ros.org/xacro">
-   <material name="red">
-        <color rgba="0.8 0 0 1"/>
-    </material>
-    <material name="green">
-        <color rgba="0 0.8 0 1"/>
-    </material>
-    <material name="blue">
-        <color rgba="0 0 0.8 1"/>
-    </material>
-    <material name="yellow">
-        <color rgba="0.8 0.8 0 1"/>
-    </material>
-    <material name="orange">
-        <color rgba="0.8 0.25 0 1"/>
-    </material>
-    <material name="black">
-        <color rgba="0 0 0 1"/>
-    </material>
-    <material name="dark_gray">
-        <color rgba="0.5 0.5 0.5 1"/>
-    </material>
-    <material name="gray">
-        <color rgba="0.753 0.753 0.753 1"/>
-    </material>
-    <material name="silver">
-        <color rgba="0.88 0.88 0.88 1"/>
-    </material>
-    <material name="white">
-        <color rgba="1 1 1 1"/>
-    </material>
+<?xml version="1.0"?>
+<robot xmlns:xacro="http://www.ros.org/wiki/xacro">
+  <!-- Colour Definitions -->
+  <material name="black">
+    <color rgba="0.0 0.0 0.0 1.0"/>
+  </material>
+  <material name="blue">
+    <color rgba="0.0 0.0 0.8 1.0"/>
+  </material>
+  <material name="green">
+    <color rgba="0.0 0.8 0.0 1.0"/>
+  </material>
+  <material name="gray">
+    <color rgba="0.753 0.753 0.753 1.0"/>
+  </material>
+  <material name="orange">
+    <color rgba="1.0 0.423529411765 0.0392156862745 1.0"/>
+  </material>
+  <material name="brown">
+    <color rgba="0.870588235294 0.811764705882 0.764705882353 1.0"/>
+  </material>
+  <material name="white">
+    <color rgba="1.0 1.0 1.0 1.0"/>
+  </material>
 </robot>

File: src/my_robot_gazebo/urdf/steer_bot.urdf.xacro (robot description, xacro)
@@ -1,24 +1,5 @@
 <?xml version="1.0"?>
-<!--
-  Robot model adapted from https://github.com/CIR-KIT/steer_drive_ros/blob/kinetic-devel/steer_drive_controller/test/common/urdf/steerbot.xacro
-  Modifications:
-    STRICTLY RESTORED: Original geometry (origins, visual, collision) from ROS 1 version.
-    Updated for ROS 2 ros2_control compatibility.
-    Removed redundant front_steer and rear_wheel macro calls.
-    Fixed 'ultramooth_mass' typo and 'ultrric_right_link' typo.
-    Cleaned up comments for strict XML parsing.
-    Removed explicit <origin> blocks from wheel_lr macro calls as origins are now internal to macros
-    to match the original ROS 1 design where origins were calculated within the macro.
-    Ensured all geometry parameters are passed correctly to macros.
-  Geometry:
-    The Ackermann steering controllers require the longitudinal
-    separation between the front and back wheel axes and the
-    lateral separation between the left and right front steering axes.
-    For this model:
-    wheel_separation_h = base_length - 2 * axle_offset = 0.4
-    wheel_separation_w = base_width + 2 * axle_offset = 0.4
--->
-<robot name="steer_bot" xmlns:xacro="http://wiki.ros.org/xacro">
-  <!-- Include xacro for wheels. wheel.xacro includes materials.xacro and inertials.xacro, so no need to include them directly here -->
+<robot name="steer_bot" xmlns:xacro="http://www.ros.org/wiki/xacro">
+  <!-- Include xacro for wheels. wheel.xacro includes materials.xacro and inertials.xacro -->
   <xacro:include filename="wheel.xacro"/>
   <xacro:arg name="use_ros2_control" default="true"/>
@@ -49,4 +30,31 @@
   <xacro:property name="camera_size" value="0.03" />
   <xacro:property name="camera_mass" value="0.1" />
+  <!-- SENSOR MACRO DEFINITION (No new file needed) -->
+  <xacro:macro name="ultrasonic_sensor" params="prefix parent xyz rpy">
+    <link name="ultrasonic_${prefix}_link">
+      <visual>
+        <origin xyz="0 0 0" rpy="0 0 0"/>
+        <geometry>
+          <box size="${ultrasonic_length} ${ultrasonic_width} ${ultrasonic_height}"/>
+        </geometry>
+        <material name="gray"/>
+      </visual>
+      <collision>
+        <origin xyz="0 0 0" rpy="0 0 0"/>
+        <geometry>
+          <box size="${ultrasonic_length} ${ultrasonic_width} ${ultrasonic_height}"/>
+        </geometry>
+      </collision>
+      <xacro:solid_cuboid_inertial
+          rpy="0 0 0" xyz="0 0 0"
+          mass="${ultrasonic_mass}"
+          x="${ultrasonic_length}" y="${ultrasonic_width}" z="${ultrasonic_height}" />
+    </link>
+    <joint name="ultrasonic_${prefix}_joint" type="fixed">
+      <parent link="${parent}"/>
+      <child link="ultrasonic_${prefix}_link"/>
+      <origin xyz="${xyz}" rpy="${rpy}"/>
+    </joint>
+  </xacro:macro>
   <!-- Base link -->
   <link name="base_link">
@@ -71,48 +79,24 @@
   <!-- Steerable front wheels -->
   <xacro:front_wheel_lr
-    name="front_right"
-    parent="base"
-    reflect="-1"
-    wheel_radius="${wheel_radius}"
-    wheel_thickness="${wheel_thickness}"
-    wheel_mass="${wheel_mass}"
-    steer_radius="${steer_radius}"
-    steer_thickness="${steer_thickness}"
-    steer_mass="${steer_mass}"
-    base_length="${base_length}"
-    base_width="${base_width}"
-    axle_offset="${axle_offset}"
-    steer_height="${wheel_radius+steer_offset}">
-  </xacro:front_wheel_lr>
+    name="front_right" parent="base" reflect="-1"
+    wheel_radius="${wheel_radius}" wheel_thickness="${wheel_thickness}" wheel_mass="${wheel_mass}"
+    steer_radius="${steer_radius}" steer_thickness="${steer_thickness}" steer_mass="${steer_mass}"
+    base_length="${base_length}" base_width="${base_width}" axle_offset="${axle_offset}"
+    steer_height="${wheel_radius+steer_offset}" />
   <xacro:front_wheel_lr
-    name="front_left"
-    parent="base"
-    reflect="1"
-    wheel_radius="${wheel_radius}"
-    wheel_thickness="${wheel_thickness}"
-    wheel_mass="${wheel_mass}"
-    steer_radius="${steer_radius}"
-    steer_thickness="${steer_thickness}"
-    steer_mass="${steer_mass}"
-    base_length="${base_length}"
-    base_width="${base_width}"
-    axle_offset="${axle_offset}"
-    steer_height="${wheel_radius+steer_offset}">
-  </xacro:front_wheel_lr>
+    name="front_left" parent="base" reflect="1"
+    wheel_radius="${wheel_radius}" wheel_thickness="${wheel_thickness}" wheel_mass="${wheel_mass}"
+    steer_radius="${steer_radius}" steer_thickness="${steer_thickness}" steer_mass="${steer_mass}"
+    base_length="${base_length}" base_width="${base_width}" axle_offset="${axle_offset}"
+    steer_height="${wheel_radius+steer_offset}" />
   <!-- Rear wheels -->
   <xacro:rear_wheel_lr
-    name="rear_right"
-    parent="base"
-    wheel_radius="${wheel_radius}"
-    wheel_thickness="${wheel_thickness}"
-    wheel_mass="${wheel_mass}">
+    name="rear_right" parent="base"
+    wheel_radius="${wheel_radius}" wheel_thickness="${wheel_thickness}" wheel_mass="${wheel_mass}">
     <origin xyz="${-base_length/2+axle_offset} ${-base_width/2-axle_offset} 0" rpy="${-90 * deg_to_rad} 0 0"/>
   </xacro:rear_wheel_lr>
   <xacro:rear_wheel_lr
-    name="rear_left"
-    parent="base"
-    wheel_radius="${wheel_radius}"
-    wheel_thickness="${wheel_thickness}"
-    wheel_mass="${wheel_mass}">
+    name="rear_left" parent="base"
+    wheel_radius="${wheel_radius}" wheel_thickness="${wheel_thickness}" wheel_mass="${wheel_mass}">
     <origin xyz="${-base_length/2+axle_offset} ${+base_width/2+axle_offset} 0" rpy="${-90 * deg_to_rad} 0 0"/>
   </xacro:rear_wheel_lr>
@@ -143,164 +127,39 @@
   </joint>
   <!-- Ultrasonic Sensor Links -->
-  <link name="ultrasonic_front_link">
-    <visual>
-      <origin xyz="0 0 0" rpy="0 0 0" />
-      <geometry>
-        <box size="${ultrasonic_length} ${ultrasonic_width} ${ultrasonic_height}" />
-      </geometry>
-      <material name="blue" />
-    </visual>
-    <collision>
-      <origin xyz="0 0 0" rpy="0 0 0" />
-      <geometry>
-        <box size="${ultrasonic_length} ${ultrasonic_width} ${ultrasonic_height}" />
-      </geometry>
-    </collision>
-    <xacro:solid_cuboid_inertial
-        rpy="0 0 0" xyz="0 0 0"
-        mass="${ultrasonic_mass}"
-        x="${ultrasonic_length}" y="${ultrasonic_width}" z="${ultrasonic_height}" />
-  </link>
-  <joint name="ultrasonic_front_joint" type="fixed">
-    <parent link="base_link"/>
-    <child link="ultrasonic_front_link"/>
-    <origin xyz="${base_length/2} 0 ${base_height/2-ultrasonic_height}" rpy="0 ${90*deg_to_rad} 0"/>
-  </joint>
-  <link name="ultrasonic_rear_link">
-    <visual>
-      <origin xyz="0 0 0" rpy="0 0 0" />
-      <geometry>
-        <box size="${ultrasonic_length} ${ultrasonic_width} ${ultrasonic_height}" />
-      </geometry>
-      <material name="blue" />
-    </visual>
-    <collision>
-      <origin xyz="0 0 0" rpy="0 0 0" />
-      <geometry>
-        <box size="${ultrasonic_length} ${ultrasonic_width} ${ultrasonic_height}" />
-      </geometry>
-    </collision>
-    <xacro:solid_cuboid_inertial
-        rpy="0 0 0" xyz="0 0 0"
-        mass="${ultrasonic_mass}"
-        x="${ultrasonic_length}" y="${ultrasonic_width}" z="${ultrasonic_height}" />
-  </link>
-  <joint name="ultrasonic_rear_joint" type="fixed">
-    <parent link="base_link"/>
-    <child link="ultrasonic_rear_link"/>
-    <origin xyz="${-base_length/2} 0 ${base_height/2-ultrasonic_height}" rpy="0 ${-90*deg_to_rad} 0"/>
-  </joint>
-  <link name="ultrasonic_right_link">
-    <visual>
-      <origin xyz="0 0 0" rpy="0 0 0" />
-      <geometry>
-        <box size="${ultrasonic_length} ${ultrasonic_width} ${ultrasonic_height}" />
-      </geometry>
-      <material name="blue" />
-    </visual>
-    <collision>
-      <origin xyz="0 0 0" rpy="0 0 0" />
-      <geometry>
-        <box size="${ultrasonic_length} ${ultrasonic_width} ${ultrasonic_height}" />
-      </geometry>
-    </collision>
-    <xacro:solid_cuboid_inertial
-        rpy="0 0 0" xyz="0 0 0"
-        mass="${ultrasonic_mass}"
-        x="${ultrasonic_length}" y="${ultrasonic_width}" z="${ultrasonic_height}" />
-  </link>
-  <joint name="ultrasonic_right_joint" type="fixed">
-    <parent link="base_link"/>
-    <child link="ultrasonic_right_link"/>
-    <origin xyz="0 ${-base_width/2} ${base_height/2-ultrasonic_height}" rpy="0 0 ${-90*deg_to_rad}"/>
-  </joint>
-  <link name="ultrasonic_left_link">
-    <visual>
-      <origin xyz="0 0 0" rpy="0 0 0" />
-      <geometry>
-        <box size="${ultrasonic_length} ${ultrasonic_width} ${ultrasonic_height}" />
-      </geometry>
-      <material name="blue" />
-    </visual>
-    <collision>
-      <origin xyz="0 0 0" rpy="0 0 0" />
-      <geometry>
-        <box size="${ultrasonic_length} ${ultrasonic_width} ${ultrasonic_height}" />
-      </geometry>
-    </collision>
-    <xacro:solid_cuboid_inertial
-        rpy="0 0 0" xyz="0 0 0"
-        mass="${ultrasonic_mass}"
-        x="${ultrasonic_length}" y="${ultrasonic_width}" z="${ultrasonic_height}" />
-  </link>
-  <joint name="ultrasonic_left_joint" type="fixed">
-    <parent link="base_link"/>
-    <child link="ultrasonic_left_link"/>
-    <origin xyz="0 ${base_width/2} ${base_height/2-ultrasonic_height}" rpy="0 0 ${90*deg_to_rad}"/>
-  </joint>
-  <!-- Colour for Gazebo (These don't define materials, they apply existing ones) -->
-  <gazebo reference="base_link">
-    <material>Gazebo/Green</material>
+  <xacro:ultrasonic_sensor prefix="front" parent="base_link" xyz="${base_length/2} 0 ${base_height/2-ultrasonic_height}" rpy="0 ${90*deg_to_rad} 0" />
+  <xacro:ultrasonic_sensor prefix="rear" parent="base_link" xyz="${-base_length/2} 0 ${base_height/2-ultrasonic_height}" rpy="0 ${-90*deg_to_rad} 0" />
+  <xacro:ultrasonic_sensor prefix="right" parent="base_link" xyz="0 ${-base_width/2} ${base_height/2-ultrasonic_height}" rpy="0 0 ${-90*deg_to_rad}" />
+  <xacro:ultrasonic_sensor prefix="left" parent="base_link" xyz="0 ${base_width/2} ${base_height/2-ultrasonic_height}" rpy="0 0 ${90*deg_to_rad}" />
+  <!-- Gazebo Plugin for ros2_control -->
+  <gazebo>
+    <plugin filename="libgazebo_ros2_control.so" name="gazebo_ros2_control">
+      <parameters>$(find my_robot_gazebo)/config/robot_controllers.yaml</parameters>
+    </plugin>
   </gazebo>
-  <gazebo reference="camera_link">
-    <material>Gazebo/Red</material>
-  </gazebo>
-  <gazebo reference="ultrasonic_front_link">
-    <material>Gazebo/Blue</material>
-  </gazebo>
-  <gazebo reference="ultrasonic_rear_link">
-    <material>Gazebo/Blue</material>
-  </gazebo>
-  <gazebo reference="ultrasonic_right_link">
-    <material>Gazebo/Blue</material>
-  </gazebo>
-  <gazebo reference="ultrasonic_left_link">
-    <material>Gazebo/Blue</material>
-  </gazebo>
-  <!-- Conditional ros2_control definition -->
-  <xacro:if value="$(arg use_ros2_control)">
-    <ros2_control name="GazeboSystem" type="system">
-      <hardware>
-        <plugin>gazebo_ros2_control/GazeboSystem</plugin>
-      </hardware>
-      <!-- Ensure these joint names EXACTLY match what your wheel.xacro creates -->
-      <joint name="front_left_steer_joint">
-        <command_interface name="position">
-          <param name="min">-0.785</param> <!-- Corresponds to max_steer_angle -->
-          <param name="max">0.785</param>
-        </command_interface>
-        <state_interface name="position" />
-        <state_interface name="velocity" />
-      </joint>
-      <joint name="front_right_steer_joint">
-        <command_interface name="position">
-          <param name="min">-0.785</param>
-          <param name="max">0.785</param>
-        </command_interface>
-        <state_interface name="position" />
-        <state_interface name="velocity" />
-      </joint>
-      <joint name="rear_left_wheel_joint">
-        <command_interface name="velocity">
-          <param name="min">-5.0</param> <!-- Example velocity limits -->
-          <param name="max">5.0</param>
-        </command_interface>
-        <state_interface name="position" />
-        <state_interface name="velocity" />
-      </joint>
-      <joint name="rear_right_wheel_joint">
-        <command_interface name="velocity">
-          <param name="min">-5.0</param>
-          <param name="max">5.0</param>
-        </command_interface>
-        <state_interface name="position" />
-        <state_interface name="velocity" />
-      </joint>
-    </ros2_control>
-    <gazebo>
-      <plugin name="gazebo_ros2_control" filename="libgazebo_ros2_control.so">
-        <robotParam>robot_description</robotParam>
-      </plugin>
-  </gazebo>
-  </xacro:if>
+  <!-- ros2_control hardware interface -->
+  <ros2_control name="GazeboSystem" type="system">
+    <hardware>
+      <plugin>gazebo_ros2_control/GazeboSystem</plugin>
+    </hardware>
+    <joint name="front_left_steer_joint">
+      <command_interface name="position"/>
+      <state_interface name="position" />
+      <state_interface name="velocity" />
+    </joint>
+    <joint name="front_right_steer_joint">
+      <command_interface name="position"/>
+      <state_interface name="position" />
+      <state_interface name="velocity" />
+    </joint>
+    <joint name="rear_left_wheel_joint">
+      <command_interface name="velocity"/>
+      <state_interface name="position" />
+      <state_interface name="velocity" />
+    </joint>
+    <joint name="rear_right_wheel_joint">
+      <command_interface name="velocity"/>
+      <state_interface name="position" />
+      <state_interface name="velocity" />
+    </joint>
+  </ros2_control>
 </robot>

Commit message: added red

File: src/my_robot_gazebo/urdf/materials.xacro (robot description, xacro)
@@ -14,4 +14,7 @@
     <color rgba="0.753 0.753 0.753 1.0"/>
   </material>
+  <material name="yellow">
+    <color rgba="0.8 0.8 0 1"/>
+  </material>
   <material name="orange">
     <color rgba="1.0 0.423529411765 0.0392156862745 1.0"/>
@@ -20,4 +23,7 @@
     <color rgba="0.870588235294 0.811764705882 0.764705882353 1.0"/>
   </material>
+  <material name="red">
+    <color rgba="0.8 0.0 0.0 1.0"/>
+  </material>
   <material name="white">
     <color rgba="1.0 1.0 1.0 1.0"/>
